File: FXAS21002_gyro.brd (EAGLE design)
At the start: 15.2 x 15.2 mm, 9 parts

Commit message: added silk
Routing:
- net INT2: track 16.4 -> 14.6 mm
Other:
- board text added: "0.1uF"
- board text added: "1.0uF"
- board text added: "100nF"
- board text added: "10k"
- board text added: "2016"
- board text added: "47k"
- board text added: "Breakout"
- board text added: "FXAS21002"
- board text added: "GND"
- board text added: "INT"
- board text added: "Laney"
- board text added: "SCL"
- board text added: "SDA"
- board text added: "VCC"
- board text added: "VIMS"
- board text added: "W&M Physics"
- board text added: "William"
- board text added: "William Laney"
- board text added: "X"
- board text added: "Y"
- board text added: "Z"
Changed lines of the file:
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@@
 <setting verticaltext="up"/>
 </settings>
-<grid distance="0.05" unitdist="inch" unit="inch" style="lines" multiple="1" display="yes" altdistance="0.025" altunitdist="inch" altunit="inch"/>
+<grid distance="0.005" unitdist="inch" unit="inch" style="lines" multiple="1" display="yes" altdistance="0.005" altunitdist="inch" altunit="inch"/>
 <layers>
 <layer number="1" name="Top" color="4" fill="1" visible="yes" active="yes"/>
@@
 <layer number="23" name="tOrigins" color="15" fill="1" visible="yes" active="yes"/>
 <layer number="24" name="bOrigins" color="15" fill="1" visible="yes" active="yes"/>
-<layer number="25" name="tNames" color="7" fill="1" visible="yes" active="yes"/>
+<layer number="25" name="tNames" color="7" fill="1" visible="no" active="yes"/>
 <layer number="26" name="bNames" color="7" fill="1" visible="no" active="yes"/>
 <layer number="27" name="tValues" color="7" fill="1" visible="no" active="yes"/>
@@
 <wire x1="15.24" y1="15.24" x2="15.24" y2="0" width="0.2032" layer="20"/>
 <wire x1="15.24" y1="0" x2="0" y2="0" width="0.2032" layer="20"/>
+<circle x="1.524" y="2.286" radius="0.127" width="0.254" layer="21"/>
+<text x="0.508" y="4.572" size="1.016" layer="21" font="vector" ratio="15">X</text>
+<text x="0.508" y="3.302" size="1.016" layer="21" font="vector" ratio="15">Y</text>
+<text x="0.508" y="1.778" size="1.016" layer="21" font="vector" ratio="15">Z</text>
+<wire x1="2.159" y1="3.556" x2="1.143" y2="3.556" width="0.254" layer="21"/>
+<wire x1="1.147296875" y1="3.586225" x2="1.528296875" y2="3.967225" width="0.254" layer="21"/>
+<wire x1="1.493234375" y1="3.184265625" x2="1.112234375" y2="3.565265625" width="0.254" layer="21"/>
+<wire x1="1.6284625" y1="4.560928125" x2="1.6284625" y2="5.576928125" width="0.254" layer="21"/>
+<wire x1="1.62785625" y1="5.557925" x2="1.24685625" y2="5.176925" width="0.254" layer="21"/>
+<wire x1="1.98819375" y1="5.17486875" x2="1.60719375" y2="5.55586875" width="0.254" layer="21"/>
+<text x="0.508" y="13.97" size="1.016" layer="21" font="vector" ratio="15">William Laney</text>
+<text x="2.54" y="1.397" size="1.016" layer="21" font="vector" ratio="15">FXAS21002</text>
+<text x="2.54" y="0.254" size="1.016" layer="21" font="vector" ratio="15">Breakout</text>
+<text x="12.827" y="13.589" size="1.016" layer="22" font="vector" ratio="15" rot="MR0">GND</text>
+<text x="12.827" y="8.509" size="1.016" layer="22" font="vector" ratio="15" rot="MR0">INT</text>
+<text x="12.827" y="5.588" size="1.016" layer="22" font="vector" ratio="15" rot="MR0">SCL</text>
+<text x="12.827" y="2.413" size="1.016" layer="22" font="vector" ratio="15" rot="MR0">SDA</text>
+<text x="12.827" y="0.635" size="1.016" layer="22" font="vector" ratio="15" rot="MR0">VCC</text>
+<text x="10.16" y="9.652" size="1.016" layer="22" font="vector" ratio="15" rot="MR0">W&amp;M Physics</text>
+<text x="10.16" y="7.62" size="1.016" layer="22" font="vector" ratio="15" rot="MR0">VIMS</text>
+<text x="5.969" y="13.843" size="1.016" layer="22" font="vector" ratio="15" rot="MR0">William</text>
+<text x="5.969" y="12.573" size="1.016" layer="22" font="vector" ratio="15" rot="MR0">Laney</text>
+<text x="8.636" y="1.651" size="1.016" layer="22" font="vector" ratio="15" rot="MR0">FXAS21002</text>
+<text x="8.636" y="0.381" size="1.016" layer="22" font="vector" ratio="15" rot="MR0">Breakout</text>
+<text x="4.826" y="7.62" size="1.016" layer="22" font="vector" ratio="15" rot="MR0">2016</text>
+<text x="12.319" y="0.254" size="1.016" layer="21" font="vector" ratio="15" rot="R90">VCC</text>
+<text x="10.668" y="7.239" size="0.8128" layer="21" font="vector" ratio="15">10k</text>
+<text x="10.668" y="3.429" size="0.8128" layer="21" font="vector" ratio="15">10k</text>
+<text x="8.255" y="12.827" size="0.8128" layer="21" font="vector" ratio="15">1.0uF</text>
+<text x="6.858" y="10.033" size="0.8128" layer="21" font="vector" ratio="15" rot="R90">0.1uF</text>
+<text x="2.286" y="12.7" size="0.8128" layer="21" font="vector" ratio="15">100nF</text>
+<text x="1.651" y="7.493" size="0.8128" layer="21" font="vector" ratio="15" rot="R90">0.1uF</text>
+<text x="8.001" y="2.921" size="0.8128" layer="21" font="vector" ratio="15" rot="R90">47k</text>
 </plain>
 <attributes>
@@
 <wire x1="13.97" y1="6.35" x2="13.705" y2="6.35" width="0.254" layer="1"/>
 <wire x1="13.705" y1="6.35" x2="11.43" y2="8.625" width="0.254" layer="1"/>
-<wire x1="8.125" y1="8.12" x2="8.39" y2="8.12" width="0.254" layer="1"/>
-<wire x1="8.39" y1="8.12" x2="10.16" y2="6.35" width="0.254" layer="1"/>
+<wire x1="10.16" y1="6.35" x2="13.97" y2="6.35" width="0.254" layer="16"/>
 <via x="10.16" y="6.35" extent="1-16" drill="0.508"/>
-<wire x1="10.16" y1="6.35" x2="13.97" y2="6.35" width="0.254" layer="16"/>
+<wire x1="8.125" y1="8.12" x2="9.025" y2="8.12" width="0.254" layer="1"/>
+<wire x1="9.025" y1="8.12" x2="10.16" y2="6.985" width="0.254" layer="1"/>
+<wire x1="10.16" y1="6.985" x2="10.16" y2="6.35" width="0.254" layer="1"/>
 </signal>
 <signal name="SDA">
@@
 <wire x1="11.43" y1="4.815" x2="11.43" y2="3.81" width="0.254" layer="1"/>
 <wire x1="11.43" y1="3.81" x2="12.33" y2="2.91" width="0.254" layer="1"/>
-<wire x1="12.7" y1="2.54" x2="13.97" y2="1.27" width="0.254" layer="1"/>
-<wire x1="6.85" y1="9.395" x2="6.85" y2="9.76" width="0.254" layer="1"/>
-<wire x1="6.85" y1="9.76" x2="7.62" y2="10.53" width="0.254" layer="1"/>
+<wire x1="12.33" y1="2.91" x2="13.97" y2="1.27" width="0.254" layer="1"/>
 <wire x1="7.62" y1="10.53" x2="9.525" y2="10.53" width="0.254" layer="1"/>
 <wire x1="9.525" y1="10.53" x2="11.325" y2="10.53" width="0.254" layer="1"/>
@@
 <wire x1="3.44" y1="2.91" x2="1.27" y2="5.08" width="0.254" layer="1"/>
 <wire x1="6.35" y1="2.91" x2="12.33" y2="2.91" width="0.254" layer="1"/>
-<wire x1="12.33" y1="2.91" x2="12.7" y2="2.54" width="0.254" layer="1"/>
+<wire x1="6.85" y1="9.395" x2="6.85" y2="10.025" width="0.254" layer="1"/>
+<wire x1="7.62" y1="10.53" x2="7.355" y2="10.53" width="0.254" layer="1"/>
+<wire x1="7.355" y1="10.53" x2="6.85" y2="10.025" width="0.254" layer="1"/>
 </signal>
 <signal name="N$1">
@@
 <signal name="INT2">
 <contactref element="U$1" pad="2"/>
-<wire x1="5.35" y1="5.845" x2="5.35" y2="5.35" width="0.254" layer="1"/>
-<wire x1="5.35" y1="5.35" x2="3.81" y2="3.81" width="0.254" layer="1"/>
-<via x="3.81" y="3.81" extent="1-16" drill="0.508"/>
+<via x="5.08" y="3.81" extent="1-16" drill="0.508"/>
 <contactref element="JP5" pad="4"/>
 <wire x1="13.97" y1="8.89" x2="10.16" y2="8.89" width="0.254" layer="16"/>
@@
 <wire x1="8.89" y1="7.62" x2="8.89" y2="5.08" width="0.254" layer="16"/>
 <wire x1="8.89" y1="5.08" x2="7.62" y2="3.81" width="0.254" layer="16"/>
-<wire x1="7.62" y1="3.81" x2="3.81" y2="3.81" width="0.254" layer="16"/>
-</signal>
-<signal name="N$2">
-<via x="10.16" y="6.35" extent="1-16" drill="0.508"/>
+<wire x1="7.62" y1="3.81" x2="5.08" y2="3.81" width="0.254" layer="16"/>
+<wire x1="5.35" y1="5.845" x2="5.35" y2="4.08" width="0.254" layer="1"/>
+<wire x1="5.35" y1="4.08" x2="5.08" y2="3.81" width="0.254" layer="1"/>
 </signal>
 </signals>
