File: FXAS21002_gyro.brd (EAGLE design)
At the start: 15.2 x 15.2 mm, 9 parts

Commit message: unified units
Parts:
- C2: value 100nF -> 0.1uF
Other:
- board text removed: "100nF"
- board text removed: "William Laney"
Changed lines of the file:
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@@
 <wire x1="1.62785625" y1="5.557925" x2="1.24685625" y2="5.176925" width="0.254" layer="21"/>
 <wire x1="1.98819375" y1="5.17486875" x2="1.60719375" y2="5.55586875" width="0.254" layer="21"/>
-<text x="0.508" y="13.97" size="1.016" layer="21" font="vector" ratio="15">William Laney</text>
+<text x="0.508" y="13.97" size="1.016" layer="21" font="vector" ratio="15">William</text>
 <text x="2.54" y="1.397" size="1.016" layer="21" font="vector" ratio="15">FXAS21002</text>
 <text x="2.54" y="0.254" size="1.016" layer="21" font="vector" ratio="15">Breakout</text>
@@
 <text x="8.255" y="12.827" size="0.8128" layer="21" font="vector" ratio="15">1.0uF</text>
 <text x="6.731" y="10.033" size="0.8128" layer="21" font="vector" ratio="15" rot="R90">0.1uF</text>
-<text x="2.286" y="12.954" size="0.8128" layer="21" font="vector" ratio="15">100nF</text>
 <text x="1.651" y="7.493" size="0.8128" layer="21" font="vector" ratio="15" rot="R90">0.1uF</text>
 <text x="8.001" y="2.921" size="0.8128" layer="21" font="vector" ratio="15" rot="R90">47k</text>
 <circle x="5.461" y="6.731" radius="0.283978125" width="0.254" layer="21"/>
 <text x="4.064" y="4.191" size="0.8128" layer="21" font="vector" ratio="15" rot="R90">FXAS21002</text>
+<text x="6.096" y="13.97" size="1.016" layer="21" font="vector" ratio="15">Laney</text>
+<text x="2.667" y="12.954" size="0.8128" layer="21" font="vector" ratio="15">0.1uF</text>
 </plain>
 <attributes>
@@
 <elements>
 <element name="C1" library="SparkFun-Passives" package="0805" value="0.1uF" x="2.54" y="8.89" rot="R90"/>
-<element name="C2" library="SparkFun-Passives" package="0805" value="100nF" x="4.445" y="12.065" rot="R180"/>
+<element name="C2" library="SparkFun-Passives" package="0805" value="0.1uF" x="4.445" y="12.065" rot="R180"/>
 <element name="C3" library="SparkFun-Passives" package="0805" value="0.1uF" x="7.62" y="11.43" rot="R90"/>
 <element name="C4" library="SparkFun-Passives" package="0805" value="1.0uF" x="9.525" y="11.43" rot="R90"/>
