File: FXAS21002_gyro.sch (EAGLE design)
At the start: 9 parts

Commit message: chnaged i2c pull up resisotr to 10k
this may not work, if that is the case its okay, I can just put a 4k7 resitor
on the board,
Parts:
- R1, R2: value 4k7 -> 10k
Changed lines of the file:
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@@
 <setting verticaltext="up"/>
 </settings>
-<grid distance="0.1" unitdist="inch" unit="inch" style="lines" multiple="1" display="yes" altdistance="0.01" altunitdist="inch" altunit="inch"/>
+<grid distance="0.1" unitdist="inch" unit="inch" style="lines" multiple="1" display="no" altdistance="0.01" altunitdist="inch" altunit="inch"/>
 <layers>
 <layer number="1" name="Top" color="4" fill="1" visible="no" active="no"/>
@@
 <part name="U$1" library="sharkdunio" deviceset="FXAS21002" device=""/>
 <part name="GND1" library="SparkFun-Aesthetics" deviceset="GND" device=""/>
-<part name="R1" library="SparkFun-Passives" deviceset="RESISTOR" device="0805-RES" value="4k7"/>
-<part name="R2" library="SparkFun-Passives" deviceset="RESISTOR" device="0805-RES" value="4k7"/>
+<part name="R1" library="SparkFun-Passives" deviceset="RESISTOR" device="0805-RES" value="10k"/>
+<part name="R2" library="SparkFun-Passives" deviceset="RESISTOR" device="0805-RES" value="10k"/>
 <part name="GND2" library="SparkFun-Aesthetics" deviceset="GND" device=""/>
 <part name="C1" library="SparkFun-Passives" deviceset="CAP" device="0805" value="0.1uF"/>

Commit message: changed int2 pin
did this to shorten trace to int2
Connections:
- net INT2: now also JP5.4; no longer JP5.5
Changed lines of the file:
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@@
 </segment>
 <segment>
-<pinref part="JP5" gate="G$1" pin="5"/>
-<wire x1="12.7" y1="99.06" x2="17.78" y2="99.06" width="0.1524" layer="91"/>
-<label x="17.78" y="99.06" size="1.27" layer="95" xref="yes"/>
+<pinref part="JP5" gate="G$1" pin="4"/>
+<wire x1="12.7" y1="96.52" x2="17.78" y2="96.52" width="0.1524" layer="91"/>
+<label x="17.78" y="96.52" size="1.27" layer="95" xref="yes"/>
 </segment>
 </net>

Commit message: unified units
Parts:
- C2: value 100nF -> 0.1uF
Changed lines of the file:
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@@
 <part name="GND2" library="SparkFun-Aesthetics" deviceset="GND" device=""/>
 <part name="C1" library="SparkFun-Passives" deviceset="CAP" device="0805" value="0.1uF"/>
-<part name="C2" library="SparkFun-Passives" deviceset="CAP" device="0805" value="100nF"/>
+<part name="C2" library="SparkFun-Passives" deviceset="CAP" device="0805" value="0.1uF"/>
 <part name="GND3" library="SparkFun-Aesthetics" deviceset="GND" device=""/>
 <part name="C3" library="SparkFun-Passives" deviceset="CAP" device="0805" value="0.1uF"/>
